Commit message: [Pokeball] Make collision geometry closer to real object.
  - replace box by sphere.

File: urdf/ur_benchmark/pokeball.urdf (robot description, URDF)
Before this commit: robot pokeball, 1 links, 0 joints
Links:
- link base_link: geometry collision sphere radius=0.025; visual mesh filename=package://hpp_practicals/meshes/ur_benchmark/pokeball.osg scale=0.025 0.025 0.025
